File: macro1.kicad_pcb (KiCad board)
At the start: 2 copper layers, 65.9 x 38.1 mm, 24 parts, among them SW1 SW_Push, U1 ATmega32U4-A, Y1 Crystal

Commit message: Trial 2: MCU Schema
Parts:
- removed C1: 1uF, Capacitor_SMD:C_0805_2012Metric
- removed C2, C3, C4: 0.1uF, Capacitor_SMD:C_0805_2012Metric
- removed C5: 10uF, Capacitor_SMD:C_0805_2012Metric
- removed C6, C7: 22pF, Capacitor_SMD:C_0805_2012Metric
- removed D1, D2, D3, D4: D_Small, Diode_SMD:D_SOD-123
- removed F1: 500mA, Fuse:Fuse_1206_3216Metric
- removed MX1, MX2, MX3, MX4: MX-NoLED, MX_Alps_Hybrid:MX-1U
- removed R1, R4: 10k, Resistor_SMD:R_0805_2012Metric
- removed R2, R3: 22, Resistor_SMD:R_0805_2012Metric
- removed SW1: SW_Push, random-keyboard-parts:SKQG-1155865
- removed U1: ATmega32U4-A, Package_QFP:TQFP-44_10x10mm_P0.8mm
- removed USB1: Molex-0548190589, random-keyboard-parts:Molex-0548190589
- removed Y1: Crystal, Crystal:Crystal_SMD_3225-4Pin_3.2x2.5mm
Routing:
- net GND: track 124.8 -> 0.00 mm, vias 4 -> 0
- net +5V: track 104.7 -> 0.00 mm, vias 8 -> 0
- net COL1: track 73.2 -> 0.00 mm, vias 2 -> 0
- net ROW0: track 70.9 -> 0.00 mm, vias 4 -> 0
- net COL0: track 53.5 -> 0.00 mm, vias 2 -> 0
- net ROW1: track 52.3 -> 0.00 mm, vias 2 -> 0
- net Net-(U1-Pad13): track 27.9 -> 0.00 mm, vias 2 -> 0
- net Net-(MX4-Pad2): track 11.9 -> 0.00 mm
- net Net-(MX2-Pad2): track 11.7 -> 0.00 mm
- net Net-(U1-Pad17): track 10.7 -> 0.00 mm
- net Net-(U1-Pad16): track 10.5 -> 0.00 mm
- net Net-(R3-Pad1): track 8.55 -> 0.00 mm, vias 2 -> 0
- net Net-(U1-Pad4): track 8.10 -> 0.00 mm, vias 2 -> 0
- net Net-(D3-Pad2): track 6.89 -> 0.00 mm
- net Net-(MX1-Pad2): track 6.61 -> 0.00 mm
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- removed copper zone on B.Cu, net GND
Other:
- board outline removed

Commit message: Trial 2: Components Layed Out
Parts:
- added C1: 0.1u, Capacitor_SMD:C_0805_2012Metric_Pad1.18x1.45mm_HandSolder, B.Cu at (136.5, 95.2)
- added C2: 0.1u, Capacitor_SMD:C_0805_2012Metric_Pad1.18x1.45mm_HandSolder, B.Cu at (145.3, 115.1)
- added C3: 0.1u, Capacitor_SMD:C_0805_2012Metric_Pad1.18x1.45mm_HandSolder, B.Cu at (132.6, 102.4)
- added C4: 0.1u, Capacitor_SMD:C_0805_2012Metric_Pad1.18x1.45mm_HandSolder, B.Cu at (150.0, 102.4)
- added C5: 10u, Capacitor_SMD:C_0805_2012Metric_Pad1.18x1.45mm_HandSolder, B.Cu at (132.6, 110.3)
- added C6: 22p, Capacitor_SMD:C_0805_2012Metric_Pad1.18x1.45mm_HandSolder, B.Cu at (154.8, 111.1)
- added C7: 22p, Capacitor_SMD:C_0805_2012Metric_Pad1.18x1.45mm_HandSolder, B.Cu at (154.8, 101.6)
- added C8: 1u, Capacitor_SMD:C_0805_2012Metric_Pad1.18x1.45mm_HandSolder, B.Cu at (141.3, 95.2)
- added D1: D, Diode_SMD:D_SOD-123, B.Cu at (176.2, 82.5)
- added D2: D, Diode_SMD:D_SOD-123, B.Cu at (179.4, 82.5)
- added D3: D, Diode_SMD:D_SOD-123, B.Cu at (176.2, 101.6)
- added D4: D, Diode_SMD:D_SOD-123, B.Cu at (179.4, 101.6)
- added F1: 500mA, Fuse:Fuse_1206_3216Metric_Pad1.42x1.75mm_HandSolder, B.Cu at (152.4, 91.3)
- added J1: AVR-ISP-6, random-keyboard-parts:Reset_Pretty-Mask, B.Cu at (131.0, 92.9)
- added R1: 22, Resistor_SMD:R_0805_2012Metric_Pad1.20x1.40mm_HandSolder, B.Cu at (149.2, 91.3)
- added R2: 22, Resistor_SMD:R_0805_2012Metric_Pad1.20x1.40mm_HandSolder, B.Cu at (144.5, 91.3)
- added R3: 10k, Resistor_SMD:R_0805_2012Metric_Pad1.20x1.40mm_HandSolder, B.Cu at (137.3, 115.1)
- added R4: 5.1k, Resistor_SMD:R_0805_2012Metric_Pad1.20x1.40mm_HandSolder, B.Cu at (151.6, 86.5)
- added R5: 5.1k, Resistor_SMD:R_0805_2012Metric_Pad1.20x1.40mm_HandSolder, B.Cu at (142.1, 86.5)
- added R6: 10k, Resistor_SMD:R_0805_2012Metric_Pad1.20x1.40mm_HandSolder, B.Cu at (129.4, 84.9)
- added SW1: Macro1, Button_Switch_Keyboard:SW_Cherry_MX_1.00u_PCB, F.Cu at (170.8, 83.8)
- added SW2: Macro2, Button_Switch_Keyboard:SW_Cherry_MX_1.00u_PCB, F.Cu at (189.9, 83.8)
- added SW3: Macro3, Button_Switch_Keyboard:SW_Cherry_MX_1.00u_PCB, F.Cu at (170.8, 102.9)
- added SW4: Macro4, Button_Switch_Keyboard:SW_Cherry_MX_1.00u_PCB, F.Cu at (189.9, 102.9)
- added SW5: PUSH_RESET, Button_Switch_SMD:SW_SPST_SKQG_WithStem, B.Cu at (135.7, 84.1)
- added U1: ATmega32U4-A, Package_QFP:TQFP-44_10x10mm_P0.8mm, B.Cu at (141.3, 106.4)
- added U2: PRTR5V0U2X, random-keyboard-parts:SOT143B, B.Cu at (146.8, 87.3)
- added USB1: HRO-TYPE-C-31-M-12, Type-C:HRO-TYPE-C-31-M-12-HandSoldering, B.Cu at (146.8, 74.0)
- added Y1: XTAL, Crystal:Crystal_SMD_3225-4Pin_3.2x2.5mm_HandSoldering, B.Cu at (156.4, 106.4)
Other:
- board outline added: 69.8 x 42.1 mm
