File: macro1.kicad_pcb (KiCad board)
At the start: 2 copper layers, 69.8 x 42.1 mm, 29 parts, among them J1 AVR-ISP-6, SW1 Macro1, SW2 Macro2, SW3 Macro3, SW4 Macro4, SW5 PUSH_RESET, U1 ATmega32U4-A, U2 PRTR5V0U2X, Y1 XTAL

Commit message: Trial 2: Finished Product
Parts:
- added FB1: 60@100MHz, Inductor_SMD:L_0805_2012Metric_Pad1.15x1.40mm_HandSolder, B.Cu at (155.6, 81.8)
- moved J1 25.4 mm to (156.4, 92.9), turned to 90 degrees
- moved C5 15.3 mm to (138.1, 96.0), turned to 0 degrees
- moved F1 9.56 mm to (142.9, 90.5)
- moved C1 8.17 mm to (132.6, 102.4), turned to -90 degrees
- moved C3 7.94 mm to (132.6, 110.3), turned to 90 degrees
- moved C8 6.35 mm to (147.6, 95.2), turned to 0 degrees
- moved R1 3.97 mm to (145.3, 91.3)
- moved R2 3.97 mm to (148.4, 91.3)
- moved Y1 1.59 mm to (154.8, 106.4)
- moved C4 1.12 mm to (150.8, 101.6), turned to 0 degrees
- moved C6 0.79 mm to (155.6, 111.1), turned to 0 degrees
- moved C7 0.79 mm to (155.6, 101.6), turned to 0 degrees
- turned R3 to 0 degrees
- turned R4 to 0 degrees
- turned R5 to 180 degrees
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Connections:
- net Net-(R1-Pad1) renamed DN
- net Net-(R2-Pad1) renamed DP
- U1 pad 10: MOSI -> MISO
- U1 pad 11: MISO -> MOSI
- U1 pad 38: ROW1 -> ROW0
- U1 pad 39: ROW0 -> ROW1
- USB1 pad 13: GND -> Earth
Routing:
- net GND: track 0.00 -> 153.9 mm, vias 0 -> 5
- net +5V: track 0.00 -> 119.4 mm, vias 0 -> 5
- net COL1: track 0.00 -> 102.1 mm, vias 0 -> 2
- net ROW1: track 0.00 -> 93.2 mm, vias 0 -> 2
- net COL0: track 0.00 -> 83.4 mm, vias 0 -> 1
- net ROW0: track 0.00 -> 82.2 mm, vias 0 -> 2
- net RESET: track 0.00 -> 55.2 mm, vias 0 -> 3
- net MOSI: track 0.00 -> 26.6 mm
- net MISO: track 0.00 -> 17.8 mm
- net VCC: track 0.00 -> 17.2 mm, vias 0 -> 2
- net SCK: track 0.00 -> 16.2 mm
- net D+: track 0.00 -> 13.4 mm
- net DP: track 0.00 -> 13.3 mm
- net XTAL1: track 0.00 -> 12.0 mm
- net XTAL2: track 0.00 -> 11.7 mm
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- added copper zone on B.Cu, net Earth
- added copper zone on F.Cu, net Earth
- added copper zone on B.Cu, net GND
- added copper zone on F.Cu, net GND
