File: _autosave-macro1.kicad_sch (KiCad schematic)
At the start: 0 parts

Commit message: Trial 2: Routed
Parts:
- added C1, C2, C3, C4: 0.1u, Capacitor_SMD:C_0805_2012Metric_Pad1.18x1.45mm_HandSolder, symbol Device:C_Small
- added C5: 10u, Capacitor_SMD:C_0805_2012Metric_Pad1.18x1.45mm_HandSolder, symbol Device:C_Small
- added C6, C7: 22p, Capacitor_SMD:C_0805_2012Metric_Pad1.18x1.45mm_HandSolder, symbol Device:C_Small
- added C8: 1u, Capacitor_SMD:C_0805_2012Metric_Pad1.18x1.45mm_HandSolder, symbol Device:C_Small
- added D1, D2, D3, D4: D, Diode_SMD:D_SOD-123, symbol Device:D
- added F1: 500mA, Fuse:Fuse_1206_3216Metric_Pad1.42x1.75mm_HandSolder, symbol Device:Polyfuse_Small
- added J1: AVR-ISP-6, random-keyboard-parts:Reset_Pretty-Mask, symbol Connector:AVR-ISP-6
- added R1, R2: 22, Resistor_SMD:R_0805_2012Metric_Pad1.20x1.40mm_HandSolder, symbol Device:R_Small
- added R3, R6: 10k, Resistor_SMD:R_0805_2012Metric_Pad1.20x1.40mm_HandSolder, symbol Device:R_Small
- added R4, R5: 5.1k, Resistor_SMD:R_0805_2012Metric_Pad1.20x1.40mm_HandSolder, symbol Device:R_Small
- added SW1: Macro1, Button_Switch_Keyboard:SW_Cherry_MX_1.00u_PCB, symbol Switch:SW_Push
- added SW2: Macro2, Button_Switch_Keyboard:SW_Cherry_MX_1.00u_PCB, symbol Switch:SW_Push
- added SW3: Macro3, Button_Switch_Keyboard:SW_Cherry_MX_1.00u_PCB, symbol Switch:SW_Push
- added SW4: Macro4, Button_Switch_Keyboard:SW_Cherry_MX_1.00u_PCB, symbol Switch:SW_Push
- added SW5: PUSH_RESET, Button_Switch_SMD:SW_SPST_SKQG_WithStem, symbol local:SW_SKQG
- added U1: ATmega32U4-A, Package_QFP:TQFP-44_10x10mm_P0.8mm, symbol MCU_Microchip_ATmega:ATmega32U4-A
- added U2: PRTR5V0U2X, random-keyboard-parts:SOT143B, symbol random-keyboard-parts:PRTR5V0U2X
- added USB1: HRO-TYPE-C-31-M-12, Type-C:HRO-TYPE-C-31-M-12-HandSoldering, symbol Type-C:HRO-TYPE-C-31-M-12
- added Y1: XTAL, Crystal:Crystal_SMD_3225-4Pin_3.2x2.5mm_HandSoldering, symbol Device:Crystal_GND24_Small
Connections:
- new net: R5.1, USB1.4 (CC1)
- new net: R3.1, U1.33 (~{HWB}/PE2)
- new net: C8.2, U1.6 (UCAP)
- new net: D4.2 (A), SW4.1
- new net: D3.2 (A), SW3.1
- new net: D1.2 (A), SW1.1
- new net: D2.2 (A), SW2.1
- new net: R4.1, USB1.10 (CC2)
- new net +5V: C1.1, C2.1, C3.1, C4.1, C5.1, F1.2, J1.2 (VCC), R6.1, U1.14 (VCC), U1.2 (UVCC), U1.24 (AVCC), U1.34 (VCC), U1.44 (AVCC), U1.7 (VBUS)
- new net COL0: SW1.2, SW3.2, U1.40 (PF1)
- new net COL1: SW2.2, SW4.2, U1.41 (PF0)
- new net D+: R2.2, U1.4 (D+)
- new net D-: R1.2, U1.3 (D-)
- new net DN: R1.1, U2.3 (IO2), USB1.5 (DN2), USB1.7 (DN1)
- new net DP: R2.1, U2.2 (IO1), USB1.6 (DP1), USB1.8 (DP2)
- new net GND: C1.2, C2.2, C3.2, C4.2, C5.2, C6.2, C7.2, C8.1, J1.6 (GND), R3.2, R4.2, R5.2, SW5.2, U1.15 (GND), U1.23 (GND), U1.35 (GND), U1.43 (GND), U1.5 (UGND), U2.1 (GND), USB1.1 (GND), USB1.12 (GND), USB1.13 (SHIELD), Y1.2, Y1.4
- new net MISO: J1.1 (MISO), U1.10 (PB2)
- new net MOSI: J1.4 (MOSI), U1.11 (PB3)
- new net RESET: J1.5 (~{RST}), R6.2, SW5.1, U1.13 (~{RESET})
- new net ROW0: D1.1 (K), D2.1 (K), U1.38 (PF5)
- new net ROW1: D3.1 (K), D4.1 (K), U1.39 (PF4)
- new net SCK: J1.3 (SCK), U1.9 (PB1)
- new net VCC: F1.1, U2.4 (VCC), USB1.11 (VBUS), USB1.2 (VBUS)
- new net XTAL1: C6.1, U1.17 (XTAL1), Y1.1
- new net XTAL2: C7.1, U1.16 (XTAL2), Y1.3
- no-connect marks 0 -> 23
