File: macro1.kicad_sch (KiCad schematic)
At the start: 24 parts, among them SW1 SW_Push, U1 ATmega32U4-A, Y1 Crystal

Commit message: First Routing: NoKeys
Connections:
- no-connect marks 0 -> 27
Changed lines of the file:
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@@
   (junction (at 107.95 53.34) (diameter 0) (color 0 0 0 0)
   )
+  (no_connect (at 96.52 98.806))
+  (no_connect (at 127 93.726))
+  (no_connect (at 127 91.186))
+  (no_connect (at 127 88.646))
+  (no_connect (at 127 86.106))
+  (no_connect (at 127 83.566))
+  (no_connect (at 127 124.206))
+  (no_connect (at 127 121.666))
+  (no_connect (at 127 119.126))
+  (no_connect (at 127 116.586))
+  (no_connect (at 127 114.046))
+  (no_connect (at 127 108.966))
+  (no_connect (at 127 106.426))
+  (no_connect (at 127 101.346))
+  (no_connect (at 127 98.806))
+  (no_connect (at 127 96.266))
+  (no_connect (at 40.386 148.59))
+  (no_connect (at 127 157.226))
+  (no_connect (at 127 154.686))
+  (no_connect (at 127 152.146))
+  (no_connect (at 127 149.606))
+  (no_connect (at 127 147.066))
+  (no_connect (at 127 144.526))
+  (no_connect (at 127 139.446))
+  (no_connect (at 127 131.826))
+  (no_connect (at 127 129.286))
+  (no_connect (at 127 126.746))
   (wire (pts (xy 88.9 121.666) (xy 88.9 123.698))
     (stroke (width 0) (type default) (color 0 0 0 0))

Commit message: First Route: NoKeys
Connections:
- net COL0: now also U1.29 (PB5)
- net COL1: now also U1.28 (PB4)
- net ROW0: now also U1.27 (PD7)
- net ROW1: now also U1.30 (PB6)
- no-connect marks 27 -> 23
Changed lines of the file:
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@@
   )
   (no_connect (at 96.52 98.806))
-  (no_connect (at 127 93.726))
-  (no_connect (at 127 91.186))
-  (no_connect (at 127 88.646))
-  (no_connect (at 127 86.106))
-  (no_connect (at 127 83.566))
+  (no_connect (at 127 108.966))
+  (no_connect (at 127 106.426))
   (no_connect (at 127 124.206))
   (no_connect (at 127 121.666))
@@
   (no_connect (at 127 116.586))
   (no_connect (at 127 114.046))
-  (no_connect (at 127 108.966))
-  (no_connect (at 127 106.426))
+  (no_connect (at 127 83.566))
+  (no_connect (at 127 91.186))
+  (no_connect (at 127 88.646))
+  (no_connect (at 127 86.106))
   (no_connect (at 127 101.346))
-  (no_connect (at 127 98.806))
-  (no_connect (at 127 96.266))
   (no_connect (at 40.386 148.59))
   (no_connect (at 127 157.226))
@@
   (no_connect (at 127 144.526))
   (no_connect (at 127 139.446))
-  (no_connect (at 127 131.826))
+  (no_connect (at 127 126.746))
   (no_connect (at 127 129.286))
-  (no_connect (at 127 126.746))
   (wire (pts (xy 88.9 121.666) (xy 88.9 123.698))
     (stroke (width 0) (type default) (color 0 0 0 0))
@@
     )
   )
+  (global_label "COL0" (shape input) (at 127 96.266 0) (fields_autoplaced)
+    (effects (font (size 1.27 1.27)) (justify left))
+    (property "Intersheet References" "${INTERSHEET_REFS}" (id 0) (at 134.2512 96.1866 0)
+      (effects (font (size 1.27 1.27)) (justify left) hide)
+    )
+  )
   (global_label "ROW1" (shape input) (at 164.084 108.966 180) (fields_autoplaced)
     (effects (font (size 1.27 1.27)) (justify right))
@@
     )
   )
+  (global_label "ROW1" (shape input) (at 127 98.806 0) (fields_autoplaced)
+    (effects (font (size 1.27 1.27)) (justify left))
+    (property "Intersheet References" "${INTERSHEET_REFS}" (id 0) (at 134.6745 98.7266 0)
+      (effects (font (size 1.27 1.27)) (justify left) hide)
+    )
+  )
+  (global_label "ROW0" (shape input) (at 127 131.826 0) (fields_autoplaced)
+    (effects (font (size 1.27 1.27)) (justify left))
+    (property "Intersheet References" "${INTERSHEET_REFS}" (id 0) (at 134.6745 131.7466 0)
+      (effects (font (size 1.27 1.27)) (justify left) hide)
+    )
+  )
+  (global_label "COL1" (shape input) (at 127 93.726 0) (fields_autoplaced)
+    (effects (font (size 1.27 1.27)) (justify left))
+    (property "Intersheet References" "${INTERSHEET_REFS}" (id 0) (at 134.2512 93.6466 0)
+      (effects (font (size 1.27 1.27)) (justify left) hide)
+    )
+  )

Commit message: Finished Product 1
Connections:
- net ROW0: no longer U1.27 (PD7)
Changed lines of the file:
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@@
-    )
-  )
-  (global_label "ROW0" (shape input) (at 127 131.826 0) (fields_autoplaced)
-    (effects (font (size 1.27 1.27)) (justify left))
-    (property "Intersheet References" "${INTERSHEET_REFS}" (id 0) (at 134.6745 131.7466 0)
-      (effects (font (size 1.27 1.27)) (justify left) hide)
     )
   )

Commit message: Trial 2: MCU Schema
Parts:
- removed C1: 1uF, Capacitor_SMD:C_0805_2012Metric, symbol Device:C_Small
- removed C2, C3, C4: 0.1uF, Capacitor_SMD:C_0805_2012Metric, symbol Device:C_Small
- removed C5: 10uF, Capacitor_SMD:C_0805_2012Metric, symbol Device:C_Small
- removed C6, C7: 22pF, Capacitor_SMD:C_0805_2012Metric, symbol Device:C_Small
- removed D1, D2, D3, D4: D_Small, Diode_SMD:D_SOD-123, symbol Device:D_Small
- removed F1: 500mA, Fuse:Fuse_1206_3216Metric, symbol Device:Polyfuse_Small
- removed MX1, MX2, MX3, MX4: MX-NoLED, MX_Alps_Hybrid:MX-1U, symbol MX_Alps_Hybrid:MX-NoLED
- removed R1, R4: 10k, Resistor_SMD:R_0805_2012Metric, symbol Device:R_Small
- removed R2, R3: 22, Resistor_SMD:R_0805_2012Metric, symbol Device:R_Small
- removed SW1: SW_Push, random-keyboard-parts:SKQG-1155865, symbol Switch:SW_Push
- removed USB1: Molex-0548190589, random-keyboard-parts:Molex-0548190589, symbol random-keyboard-parts:Molex-0548190589
- removed Y1: Crystal, Crystal:Crystal_SMD_3225-4Pin_3.2x2.5mm, symbol Device:Crystal_GND24_Small
- added C? (x4): 0.1u, symbol Device:C_Small
- added C? (x2): 22p, symbol Device:C_Small
- added C?: C_Small, symbol Device:C_Small
- added C?: 10u, symbol Device:C_Small
- added F?: 500mA, symbol Device:Polyfuse_Small
- added J?: AVR-ISP-6, symbol Connector:AVR-ISP-6
- added R? (x2): 5.1k, symbol Device:R_Small
- added R? (x2): 22, symbol Device:R_Small
- added R? (x2): 10k, symbol Device:R_Small
- added SW?: PUSH_RESET, symbol local:SW_SKQG
- added U?: PRTR5V0U2X, symbol random-keyboard-parts:PRTR5V0U2X
- added USB?: HRO-TYPE-C-31-M-12, symbol Type-C:HRO-TYPE-C-31-M-12
- added Y?: XTAL, symbol Device:Crystal_GND24_Small
Connections:
- net +5V: now also C?.1, C?.1, C?.1, C?.1, C?.1, F?.2, J?.2 (VCC), R?.1
- net D+: now also U1.4 (D+), R?.2
- net D-: now also U1.3 (D-), R?.2
- net GND: now also C?.1, C?.2, C?.2, C?.2, C?.2, C?.2, C?.2, C?.2, J?.6 (GND), R?.2, R?.2, R?.2, SW?.2, U?.1 (GND), USB?.1 (GND), USB?.12 (GND), USB?.13 (SHIELD), Y?.2, Y?.4
- net VCC: now also F?.1, U?.4 (VCC), USB?.11 (VBUS), USB?.2 (VBUS)
- net at U1.33 (~{HWB}/PE2): now also R?.1
- net XTAL1: now reaches U1.17 (XTAL1)
- net XTAL1: now also C?.1, Y?.1
- net XTAL2: now reaches U1.16 (XTAL2)
- net XTAL2: now also C?.1, Y?.3
- net at U1.6 (UCAP): now also C?.2
- net MOSI: now reaches U1.10 (PB2)
- net MOSI: now also J?.4 (MOSI)
- net MISO: now reaches U1.11 (PB3)
- net MISO: now also J?.1 (MISO)
- net SCK: now reaches U1.9 (PB1)
- net SCK: now also J?.3 (SCK)
- net COL0: no longer names the net of U1.29 (PB5)
- net COL1: no longer names the net of U1.28 (PB4)
- net ROW1: no longer names the net of U1.30 (PB6)
- new net: R?.1, USB?.4 (CC1)
- new net: R?.1, U?.2 (IO1), USB?.6 (DP1), USB?.8 (DP2)
- new net: R?.1, U?.3 (IO2), USB?.5 (DN2), USB?.7 (DN1)
- new net: R?.1, USB?.10 (CC2)
- new net RESET: J?.5 (~{RST}), R?.2, SW?.1
- no-connect marks 23 -> 5

Commit message: Trial 2: Final Schema
Parts:
- added D1, D2, D3, D4: D, Diode_SMD:D_SOD-123, symbol Device:D
- added SW1: Macro1, MX_Alps_Hybrid:MX-1U, symbol Switch:SW_Push
- added SW2: Macro2, MX_Alps_Hybrid:MX-1U, symbol Switch:SW_Push
- added SW3: Macro3, MX_Alps_Hybrid:MX-1U, symbol Switch:SW_Push
- added SW4: Macro4, MX_Alps_Hybrid:MX-1U, symbol Switch:SW_Push
- C1, C2, C3, C4, C5, C6, C7, C8: renamed from C?; footprint (none) -> Capacitor_SMD:C_0805_2012Metric_Pad1.18x1.45mm_HandSolder
- F1: renamed from F?; footprint (none) -> Fuse:Fuse_1206_3216Metric_Pad1.42x1.75mm_HandSolder
- J1: renamed from J?; footprint (none) -> random-keyboard-parts:Reset_Pretty-Mask
- R1, R2, R3, R4, R5, R6: renamed from R?; footprint (none) -> Resistor_SMD:R_0805_2012Metric_Pad1.20x1.40mm_HandSolder
- SW5: renamed from SW?; footprint (none) -> Button_Switch_SMD:SW_SPST_SKQG_WithStem
- U2: renamed from U?; footprint (none) -> random-keyboard-parts:SOT143B
- USB1: renamed from USB?; footprint (none) -> Type-C:HRO-TYPE-C-31-M-12-HandSoldering
- Y1: renamed from Y?; footprint (none) -> Crystal:Crystal_SMD_3225-4Pin_3.2x2.5mm_HandSoldering
Connections:
- net ROW1: now reaches U1.38 (PF5)
- net ROW1: now also D3.1 (K), D4.1 (K)
- net ROW0: now reaches U1.39 (PF4)
- net ROW0: now also D1.1 (K), D2.1 (K)
- net COL0: now reaches U1.40 (PF1)
- net COL0: now also SW1.2, SW3.2
- net COL1: now reaches U1.41 (PF0)
- net COL1: now also SW2.2, SW4.2
- new net: D4.2 (A), SW4.1
- new net: D3.2 (A), SW3.1
- new net: D1.2 (A), SW1.1
- new net: D2.2 (A), SW2.1
- no-connect marks 5 -> 24
Other:
- moved on the sheet: F1, R1, R2, R4, R5, U2, USB1

Commit message: Trial 2: Components Layed Out
Parts:
- C8: value C_Small -> 1u
- SW1, SW2, SW3, SW4: footprint MX_Alps_Hybrid:MX-1U -> Button_Switch_Keyboard:SW_Cherry_MX_1.00u_PCB
Connections:
- net RESET: now also U1.13 (~{RESET})
- no-connect marks 24 -> 23
Changed lines of the file:
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@@
   (no_connect (at 155.448 61.722))
   (no_connect (at 155.448 51.562))
-  (no_connect (at 124.968 51.562))
   (no_connect (at 155.448 82.042))
   (no_connect (at 155.448 76.962))
@@
     (property "Intersheet References" "${INTERSHEET_REFS}" (id 0) (at 94.1546 56.5996 90)
       (effects (font (size 1.27 1.27)) (justify left) hide)
+    )
+  )
+  (global_label "RESET" (shape input) (at 124.968 51.562 180) (fields_autoplaced)
+    (effects (font (size 1.27 1.27)) (justify right))
+    (property "Intersheet References" "${INTERSHEET_REFS}" (id 0) (at 116.8097 51.4826 0)
+      (effects (font (size 1.27 1.27)) (justify right) hide)
     )
   )
@@
     (property "Reference" "SW4" (id 0) (at 243.84 94.234 0))
     (property "Value" "Macro4" (id 1) (at 243.84 96.774 0))
-    (property "Footprint" "MX_Alps_Hybrid:MX-1U" (id 2) (at 243.84 96.774 0)
+    (property "Footprint" "Button_Switch_Keyboard:SW_Cherry_MX_1.00u_PCB" (id 2) (at 243.84 96.774 0)
       (effects (font (size 1.27 1.27)) hide)
     )
@@
     (property "Reference" "SW1" (id 0) (at 228.6 73.914 0))
     (property "Value" "Macro1" (id 1) (at 228.6 76.454 0))
-    (property "Footprint" "MX_Alps_Hybrid:MX-1U" (id 2) (at 228.6 76.454 0)
+    (property "Footprint" "Button_Switch_Keyboard:SW_Cherry_MX_1.00u_PCB" (id 2) (at 228.6 76.454 0)
       (effects (font (size 1.27 1.27)) hide)
     )
@@
     (property "Reference" "SW3" (id 0) (at 228.6 94.234 0))
     (property "Value" "Macro3" (id 1) (at 228.6 96.774 0))
-    (property "Footprint" "MX_Alps_Hybrid:MX-1U" (id 2) (at 228.6 96.774 0)
+    (property "Footprint" "Button_Switch_Keyboard:SW_Cherry_MX_1.00u_PCB" (id 2) (at 228.6 96.774 0)
       (effects (font (size 1.27 1.27)) hide)
     )
@@
     (in_bom yes) (on_board yes)
     (property "Reference" "C8" (id 0) (at 117.602 82.042 90))
-    (property "Value" "C_Small" (id 1) (at 120.396 87.122 90))
+    (property "Value" "1u" (id 1) (at 120.396 87.122 90))
     (property "Footprint" "Capacitor_SMD:C_0805_2012Metric_Pad1.18x1.45mm_HandSolder" (id 2) (at 117.602 84.582 0)
       (effects (font (size 1.27 1.27)) hide)
@@
     (property "Reference" "SW2" (id 0) (at 243.84 73.914 0))
     (property "Value" "Macro2" (id 1) (at 243.84 76.454 0))
-    (property "Footprint" "MX_Alps_Hybrid:MX-1U" (id 2) (at 243.84 76.454 0)
+    (property "Footprint" "Button_Switch_Keyboard:SW_Cherry_MX_1.00u_PCB" (id 2) (at 243.84 76.454 0)
       (effects (font (size 1.27 1.27)) hide)
     )
@@
     )
     (path "/c5a6deb0-d504-493b-8609-390e9df1df35"
-      (reference "C8") (unit 1) (value "C_Small") (footprint "Capacitor_SMD:C_0805_2012Metric_Pad1.18x1.45mm_HandSolder")
+      (reference "C8") (unit 1) (value "1u") (footprint "Capacitor_SMD:C_0805_2012Metric_Pad1.18x1.45mm_HandSolder")
     )
     (path "/ab5a145f-a44a-4fc1-88b5-81f18910d6e8"
@@
     )
     (path "/533b9a83-b527-4173-9434-44aa9b5be45b"
-      (reference "SW1") (unit 1) (value "Macro1") (footprint "MX_Alps_Hybrid:MX-1U")
+      (reference "SW1") (unit 1) (value "Macro1") (footprint "Button_Switch_Keyboard:SW_Cherry_MX_1.00u_PCB")
     )
     (path "/dbb8df32-6d71-41e2-a015-d59534da8431"
-      (reference "SW2") (unit 1) (value "Macro2") (footprint "MX_Alps_Hybrid:MX-1U")
+      (reference "SW2") (unit 1) (value "Macro2") (footprint "Button_Switch_Keyboard:SW_Cherry_MX_1.00u_PCB")
     )
     (path "/6eaa9de2-0a7d-4d4f-ae17-46fea089947f"
-      (reference "SW3") (unit 1) (value "Macro3") (footprint "MX_Alps_Hybrid:MX-1U")
+      (reference "SW3") (unit 1) (value "Macro3") (footprint "Button_Switch_Keyboard:SW_Cherry_MX_1.00u_PCB")
     )
     (path "/38c76b3b-9112-45ed-8e38-2ff88a5ae0af"
-      (reference "SW4") (unit 1) (value "Macro4") (footprint "MX_Alps_Hybrid:MX-1U")
+      (reference "SW4") (unit 1) (value "Macro4") (footprint "Button_Switch_Keyboard:SW_Cherry_MX_1.00u_PCB")
     )
     (path "/538c0ba3-cf2d-4f48-b095-701bcb8fd997"

Commit message: Trial 2: Routed
Connections:
- net DP: now reaches R2.1, U2.2 (IO1), USB1.6 (DP1), USB1.8 (DP2)
- net DN: now reaches R1.1, U2.3 (IO2), USB1.5 (DN2), USB1.7 (DN1)
Changed lines of the file:
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@@
+    )
+  )
+  (global_label "DP" (shape input) (at 54.102 101.346 270) (fields_autoplaced)
+    (effects (font (size 1.27 1.27)) (justify right))
+    (property "Intersheet References" "${INTERSHEET_REFS}" (id 0) (at 54.0226 106.2991 90)
+      (effects (font (size 1.27 1.27)) (justify right) hide)
     )
   )
@@
     )
   )
+  (global_label "DN" (shape input) (at 54.102 98.806 90) (fields_autoplaced)
+    (effects (font (size 1.27 1.27)) (justify left))
+    (property "Intersheet References" "${INTERSHEET_REFS}" (id 0) (at 54.0226 93.7924 90)
+      (effects (font (size 1.27 1.27)) (justify left) hide)
+    )
+  )

Commit message: Trial 2: Finished Product
Parts:
- added FB1: 60@100MHz, symbol Device:FerriteBead_Small
Connections:
- net GND: now also FB1.2; no longer USB1.13 (SHIELD)
- net MISO: now also U1.10 (PB2); no longer U1.11 (PB3)
- net MOSI: now also U1.11 (PB3); no longer U1.10 (PB2)
- net ROW0: now also U1.38 (PF5); no longer U1.39 (PF4)
- net ROW1: now also U1.39 (PF4); no longer U1.38 (PF5)
- new net Earth: FB1.1, USB1.13 (SHIELD)
Other:
- moved on the sheet: R6, SW5
