File: _autosave-macro1.kicad_pcb (KiCad board)
At the start: 2 copper layers, 69.8 x 42.1 mm, 29 parts, among them J1 AVR-ISP-6, SW1 Macro1, SW2 Macro2, SW3 Macro3, SW4 Macro4, SW5 PUSH_RESET, U1 ATmega32U4-A, U2 PRTR5V0U2X, Y1 XTAL

Commit message: Trial 2: Finished Product
Parts:
- added FB1: 60@100MHz, Inductor_SMD:L_0805_2012Metric_Pad1.15x1.40mm_HandSolder, B.Cu at (155.6, 81.8)
Connections:
- USB1 pad 13: GND -> Earth
Routing:
- net GND: track 136.2 -> 153.9 mm
- net Earth: vias 0 -> 4
- added copper zone on B.Cu, net Earth
- added copper zone on F.Cu, net Earth

Commit message: MOSI Fix
Connections:
- U1 pad 10: MISO -> MOSI
- U1 pad 11: MOSI -> MISO
Routing:
- net MOSI: track 26.6 -> 20.4 mm
- net MISO: track 17.8 -> 17.3 mm
